File: pcb/pcb.kicad_pcb (KiCad board)
At the start: 2 copper layers, 40 parts

Commit message: feat: schematic for full adder mostly done
Parts:
- removed B_REG_1_9, B_REG_9_17: SN74HC574N, 74hc:20pdip
- removed B_REG_TXRX_1_9, B_REG_TXRX_9_17: SN74HC245N, 74hc:20pdip
- added B_REG_1_8: SN74HC574N, 74hc:20pdip, F.Cu at (113.9, 129.8)
- added B_REG_9_16: SN74HC574N, 74hc:20pdip, F.Cu at (169.4, 129.8)
- added B_REG_TXRX_1_8: SN74HC245N, 74hc:20pdip, F.Cu at (114.0, 174.4)
- added B_REG_TXRX_9_16: SN74HC245N, 74hc:20pdip, F.Cu at (169.6, 174.4)
- added FULL_ADDER_13_16: CD74HC283E, 74hc:16pdip, F.Cu at (272.6, 184.6)
- added FULL_ADDER_1_4: CD74HC283E, 74hc:16pdip, F.Cu at (283.2, 184.6)
- added FULL_ADDER_5_8: CD74HC283E, 74hc:16pdip, F.Cu at (293.7, 184.6)
- added FULL_ADDER_9_12: CD74HC283E, 74hc:16pdip, F.Cu at (304.3, 184.6)
- added FULL_ADDER_TXRX_1_8: SN74HC245N, 74hc:20pdip, F.Cu at (261.6, 135.2)
- added FULL_ADDER_TXRX_9_16: SN74HC245N, 74hc:20pdip, F.Cu at (272.2, 135.2)
- added NAND_13_16: SN74HC00N, 74hc:14pdip, F.Cu at (314.9, 183.3)
- added NAND_1_4: SN74HC00N, 74hc:14pdip, F.Cu at (325.5, 183.3)
- added NAND_5_8: SN74HC00N, 74hc:14pdip, F.Cu at (336.1, 183.3)
- added NAND_9_12: SN74HC00N, 74hc:14pdip, F.Cu at (346.6, 183.3)
- moved B_1 200.0 mm to (102.4, 145.6), turned to 180 degrees
- moved B_2 192.3 mm to (109.4, 145.6), turned to 180 degrees
- moved B_3 184.9 mm to (116.3, 145.6), turned to 180 degrees
- moved B_6 178.6 mm to (134.3, 145.6)
- moved B_4 177.8 mm to (123.1, 145.6), turned to 180 degrees
- moved B_5 173.5 mm to (127.4, 145.6)
- moved B_7 170.3 mm to (141.2, 145.6)
- moved B_8 162.3 mm to (148.0, 145.6)
- moved B_9 151.4 mm to (157.9, 145.6), turned to 180 degrees
- moved B_10 143.9 mm to (164.8, 145.6), turned to 180 degrees
- moved B_13 138.9 mm to (182.8, 145.6)
- moved B_11 136.9 mm to (171.5, 145.6), turned to 180 degrees
- moved B_14 130.2 mm to (189.8, 145.6)
- moved B_12 130.0 mm to (178.5, 145.6), turned to 180 degrees
- moved B_15 121.8 mm to (196.6, 145.6)
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Routing:
- net GND: track 79.3 -> 158.5 mm
- net /B_9: track 0.00 -> 67.6 mm
- net /B_1: track 0.00 -> 67.6 mm
- net /B_16: track 0.00 -> 67.1 mm
- net /B_8: track 0.00 -> 67.1 mm
- net /B_10: track 0.00 -> 59.6 mm
- net /B_2: track 0.00 -> 59.6 mm
- net /B_15: track 0.00 -> 58.8 mm
- net /B_7: track 0.00 -> 58.8 mm
- net /B_11: track 0.00 -> 50.8 mm
- net /B_3: track 0.00 -> 50.8 mm
- net /B_14: track 0.00 -> 50.1 mm
- net /B_6: track 0.00 -> 50.1 mm
- net /B_12: track 0.00 -> 42.3 mm
- net /B_4: track 0.00 -> 42.3 mm
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